File: esp32s2-uart.sch (KiCad schematic (older format))
At the start: 9 parts

Commit message: updata
Parts:
- added C? (x3): 2.2uf, Capacitor_SMD:C_0603_1608Metric, symbol Device:C
- added C?: 0.1uf, Capacitor_SMD:C_0402_1005Metric, symbol Device:C
- added D? (x4): PESD3V3L4UF, Package_TO_SOT_SMD:SOT-886, symbol Power_Protection:PESD3V3L4UF
- added D? (x2): ESD9B3.3ST5G, Diode_SMD:D_SOD-923, symbol Diode:ESD9B3.3ST5G
- added J?: Conn_02x04_Odd_Even, symbol Connector_Generic:Conn_02x04_Odd_Even
- added R? (x2): 22, Resistor_SMD:R_0402_1005Metric, symbol Device:R
- added R?: 0, Resistor_SMD:R_0402_1005Metric, symbol Device:R
- added R?: NC, Resistor_SMD:R_0402_1005Metric, symbol Device:R
- added RN?: 2.2k, Resistor_SMD:R_Array_Concave_4x0402, symbol Device:R_Pack04
- added TP?: TXD, symbol Connector:TestPoint
- added TP?: RXD, symbol Connector:TestPoint
- added TP?: IO0, symbol Connector:TestPoint
- added TP?: EN, symbol Connector:TestPoint
- C?: value C -> 0.1uf; footprint (none) -> Capacitor_SMD:C_0402_1005Metric
- R?: value R -> 10k; footprint (none) -> Resistor_SMD:R_0402_1005Metric
Connections:
- net labels added: +3.3V, +5V, EN, GND, IO0, UART_RX, UART_TX, USB_D+, USB_D-, VOUT
- wire segments 0 -> 44
- no-connect marks 0 -> 4
Other:
- moved on the sheet: C?, D?, R?

Commit message: add esp32-s2fh4 symbol lib
Parts:
- removed U?: ESP32-S2-WROVER, RF_Module:ESP32-S2-WROVER, symbol RF_Module:ESP32-S2-WROVER
- added U?: ESP32-S2FH4, Package_DFN_QFN:QFN-56-1EP_7x7mm_P0.4mm_EP5.6x5.6mm, symbol mylib:ESP32-S2FH4
Connections:
- wire segments 44 -> 46
Other:
- moved on the sheet: C?, D?, J?, R?, TP?, U?

Commit message: complete schematic
Parts:
- removed TP?: TXD, symbol Connector:TestPoint
- removed TP?: RXD, symbol Connector:TestPoint
- removed TP?: IO0, symbol Connector:TestPoint
- removed TP?: EN, symbol Connector:TestPoint
- added AE1: Antenna_Chip, RF_Antenna:Johanson_2450AT43F0100, symbol Device:Antenna_Chip
- added C10, C8: TBD, Capacitor_SMD:C_0402_1005Metric, symbol Device:C
- added C11, C12, C13, C14, C5, C7, C9: 0.1uf, Capacitor_SMD:C_0402_1005Metric, symbol Device:C
- added D3: LED, LED_SMD:LED_0603_1608Metric, symbol Device:LED
- added J2: Conn_01x06, Connector_PinHeader_1.27mm:PinHeader_1x06_P1.27mm_Vertical, symbol Connector_Generic:Conn_01x06
- added L1: L, Inductor_SMD:L_0402_1005Metric, symbol Device:L
- added R3: 1k, Resistor_SMD:R_0402_1005Metric, symbol Device:R
- added R5: 10k, Resistor_SMD:R_0402_1005Metric, symbol Device:R
- added Y1: Crystal_GND24_Small, Crystal:Crystal_SMD_EuroQuartz_MT-4Pin_3.2x2.5mm, symbol Device:Crystal_GND24_Small
- C1, C4: renamed from C?; value 2.2uf -> 10uf
- C2: renamed from C?; value 2.2uf -> 4.7uf
- D5, D6, D7, D8: renamed from D?; footprint (none) -> LED_SMD:LED_0603_1608Metric
- J1: renamed from J?; footprint (none) -> Connector_USB:USB_C_Receptacle_Palconn_UTC16-G
- J3: renamed from J?; footprint (none) -> Connector_PinHeader_2.54mm:PinHeader_2x04_P2.54mm_Horizontal
- gave numbers to parts that had none: 13
Connections:
- net labels added: CTS, DBG_EN, DBG_IO0, DBG_RX, DBG_TX, LNA_IN, RTS
- wire segments 46 -> 85
- no-connect marks 4 -> 34
Other:
- moved on the sheet: C3, C4

Commit message: update
Parts:
- removed D2: ESD9B3.3ST5G, Diode_SMD:D_SOD-923, symbol Diode:ESD9B3.3ST5G
- removed D4: PESD3V3L4UF, Package_TO_SOT_SMD:SOT-886, symbol Power_Protection:PESD3V3L4UF
- removed D5, D6: LED, LED_SMD:LED_0603_1608Metric, symbol Device:LED
- removed J3: Conn_02x04_Odd_Even, Connector_PinHeader_2.54mm:PinHeader_2x04_P2.54mm_Horizontal, symbol Connector_Generic:Conn_02x04_Odd_Even
- removed R6: 0, Resistor_SMD:R_0402_1005Metric, symbol Device:R
- removed R7: NC, Resistor_SMD:R_0402_1005Metric, symbol Device:R
- removed RN1: 2.2k, Resistor_SMD:R_Array_Concave_4x0402, symbol Device:R_Pack04
- added C10, C8: 10pf, Capacitor_SMD:C_0402_1005Metric, symbol Device:C
- added D1: RED, LED_SMD:LED_0603_1608Metric, symbol Device:LED
- added D2: GREEN, LED_SMD:LED_0603_1608Metric, symbol Device:LED
- added D4, D5, D6, D8, D9: PESD5V0S1BA, Diode_SMD:D_SOD-323, symbol Diode:ESD9B3.3ST5G
- added J3: Conn_02x05_Counter_Clockwise, my_footprint:Header_2x5_pin, symbol Connector_Generic:Conn_02x05_Counter_Clockwise
- added R3, R4, R8, R9: 1k, Resistor_SMD:R_0402_1005Metric, symbol Device:R
- added SW1: SW_Push, Button_Switch_SMD:SW_SPST_B3U-3000P-B, symbol Switch:SW_Push
- added U2: USBLC6-2SC6, Package_TO_SOT_SMD:SOT-23-6, symbol Power_Protection:USBLC6-2SC6
- C2: value 4.7uf -> 10uf
- D3: value LED -> BLUE
- D7: renamed from D1; value ESD9B3.3ST5G -> PESD5V0S1BA; footprint Diode_SMD:D_SOD-923 -> Diode_SMD:D_SOD-323
- J1: renamed from J2; footprint Connector_PinHeader_1.27mm:PinHeader_1x06_P1.27mm_Vertical -> Connector_PinHeader_1.00mm:PinHeader_1x06_P1.00mm_Vertical
- J2: renamed from J1; symbol Connector:USB_C_Receptacle_USB2.0 -> esp32s2-uart-rescue:USB_C_Receptacle_USB2.0-Connector
- renumbered C8 to C15, C10 to C16, C4 to C3, C3 to C4, D7 to D10, D8 to D11, R3 to R5, R4 to R6, R5 to R7, U2 to U3
Connections:
- net labels added: CTS_TDI, EN_TCK, IO0_TMS, RTS_TDO
- net labels removed: CTS, EN, IO0, RTS, VOUT
- wire segments 85 -> 110
- no-connect marks 34 -> 32
Other:
- moved on the sheet: AE1, C1, C11, C12, C13, C14, C15, C16, C2, C3, C4, C5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

Commit message: update
Parts:
- removed J1: Conn_01x06, Connector_PinHeader_1.00mm:PinHeader_1x06_P1.00mm_Vertical, symbol Connector_Generic:Conn_01x06
- added TP1, TP2, TP3, TP4, TP5, TP6: TestPoint, TestPoint:TestPoint_Pad_D1.0mm, symbol Connector:TestPoint
Connections:
- net +3V3: now also TP2.1
- net DBG_EN: now also TP4.1
- net DBG_IO0: now also TP3.1
- net DBG_RX: now also TP6.1
- net DBG_TX: now also TP5.1
- net GND: now also TP1.1
Changed lines of the file:
@@
 	0    1    1    0
-$EndComp
-$Comp
-L Connector_Generic:Conn_01x06 J1
-U 1 1 60624C02
-P 800 4950
-F 0 "J1" H 718 4425 50  0000 C CNN
-F 1 "Conn_01x06" H 718 4516 50  0000 C CNN
-F 2 "Connector_PinHeader_1.00mm:PinHeader_1x06_P1.00mm_Vertical" H 800 4950 50  0001 C CNN
-F 3 "~" H 800 4950 50  0001 C CNN
-	1    800  4950
-	-1   0    0    1
 $EndComp
 Text Label 4650 3750 0    50   ~ 0
@@
 Wire Wire Line
 	10800 4750 10800 5350
+$Comp
+L Connector:TestPoint TP1
+U 1 1 61E1E1B1
+P 1000 4650
+F 0 "TP1" V 1000 4900 50  0000 C CNN
+F 1 "TestPoint" V 1104 4722 50  0001 C CNN
+F 2 "TestPoint:TestPoint_Pad_D1.0mm" H 1200 4650 50  0001 C CNN
+F 3 "~" H 1200 4650 50  0001 C CNN
+	1    1000 4650
+	0    -1   -1   0
+$EndComp
+$Comp
+L Connector:TestPoint TP2
+U 1 1 61E2A09D
+P 1000 4750
+F 0 "TP2" V 1000 5000 50  0000 C CNN
+F 1 "TestPoint" V 1104 4822 50  0001 C CNN
+F 2 "TestPoint:TestPoint_Pad_D1.0mm" H 1200 4750 50  0001 C CNN
+F 3 "~" H 1200 4750 50  0001 C CNN
+	1    1000 4750
+	0    -1   -1   0
+$EndComp
+$Comp
+L Connector:TestPoint TP3
+U 1 1 61E2A21B
+P 1000 4850
+F 0 "TP3" V 1000 5100 50  0000 C CNN
+F 1 "TestPoint" V 1104 4922 50  0001 C CNN
+F 2 "TestPoint:TestPoint_Pad_D1.0mm" H 1200 4850 50  0001 C CNN
+F 3 "~" H 1200 4850 50  0001 C CNN
+	1    1000 4850
+	0    -1   -1   0
+$EndComp
+$Comp
+L Connector:TestPoint TP4
+U 1 1 61E2A3F7
+P 1000 4950
+F 0 "TP4" V 1000 5200 50  0000 C CNN
+F 1 "TestPoint" V 1104 5022 50  0001 C CNN
+F 2 "TestPoint:TestPoint_Pad_D1.0mm" H 1200 4950 50  0001 C CNN
+F 3 "~" H 1200 4950 50  0001 C CNN
+	1    1000 4950
+	0    -1   -1   0
+$EndComp
+$Comp
+L Connector:TestPoint TP5
+U 1 1 61E2A5CE
+P 1000 5050
+F 0 "TP5" V 1000 5300 50  0000 C CNN
+F 1 "TestPoint" V 1104 5122 50  0001 C CNN
+F 2 "TestPoint:TestPoint_Pad_D1.0mm" H 1200 5050 50  0001 C CNN
+F 3 "~" H 1200 5050 50  0001 C CNN
+	1    1000 5050
+	0    -1   -1   0
+$EndComp
+$Comp
+L Connector:TestPoint TP6
+U 1 1 61E2A7E9
+P 1000 5150
+F 0 "TP6" V 1000 5400 50  0000 C CNN
+F 1 "TestPoint" V 1104 5222 50  0001 C CNN
+F 2 "TestPoint:TestPoint_Pad_D1.0mm" H 1200 5150 50  0001 C CNN
+F 3 "~" H 1200 5150 50  0001 C CNN
+	1    1000 5150
+	0    -1   -1   0
+$EndComp
 $EndSCHEMATC

Commit message: v1.0
Parts:
- removed D4, D5, D6, D7, D8, D9: PESD5V0S1BA, Diode_SMD:D_SOD-323, symbol Diode:ESD9B3.3ST5G
- added D4, D5: PESD5V0L5UY, Package_TO_SOT_SMD:SOT-363_SC-70-6, symbol Power_Protection:PESD5V0L5UY
- added J1: USB_A, Connector_USB:USB_A_CNCTech_1001-011-01101_Horizontal, symbol Connector:USB_A
- J2: footprint Connector_USB:USB_C_Receptacle_Palconn_UTC16-G -> my_footprint:USB_C_Receptacle; symbol esp32s2-uart-rescue:USB_C_Receptacle_USB2.0-Connector -> Connector:USB_C_Receptacle_USB2.0
- SW1: footprint Button_Switch_SMD:SW_SPST_B3U-3000P-B -> my_footprint:button
Connections:
- net +3V3: now also D4.4 (K3)
- net +5V: now also D4.6 (K5), J1.1 (VBUS)
- net CTS_TDI: now also U3.40 (GPIO36), D4.3 (K2); no longer U3.37 (GPIO33)
- net EN_TCK: now also U3.39 (GPIO35), D5.6 (K5); no longer U3.41 (GPIO37)
- net GND: now also D4.1 (K1), D5.1 (K1), J1.4 (GND), J1.5 (Shield)
- net IO0_TMS: now also D5.3 (K2)
- net RTS_TDO: now also D4.5 (K4)
- net UART_RX: now also U3.41 (GPIO37), D5.5 (K4); no longer U3.40 (GPIO36)
- net UART_TX: now also U3.43 (MTCK), D5.4 (K3); no longer U3.39 (GPIO35)
- net USB_D+: now also J2.A6 (D+), J2.B6 (D+), U2.3 (I/O2), J1.3 (D+); no longer R2.1, U3.26 (GPIO20)
- net USB_D-: now also J2.A7 (D-), J2.B7 (D-), U2.1 (I/O1), J1.2 (D-); no longer R1.1, U3.25 (GPIO19)
- new net: R1.1, U3.25 (GPIO19)
- new net: R2.1, U3.26 (GPIO20)
- no-connect marks 32 -> 34
Other:
- moved on the sheet: C10, C11, C12, C13, C14, C3, C4, C5, C6, C7, C8, C9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

Commit message: v1.0
Parts:
- added logo1: logo, my_footprint:ESP-USB-Bridge, symbol Mechanical:MountingHole
- D10, D11: value LED -> LED_YELLOW
Connections:
- net +3V3: now also D10.2 (A), D11.2 (A), J3.5 (Pin_5); no longer D4.4 (K3), J3.4 (Pin_4)
- net +5V: no longer D10.2 (A), D11.2 (A), D4.6 (K5), J3.5 (Pin_5)
- net GND: no longer J3.7 (Pin_7)
- net TMS: now reaches U3.37 (GPIO33)
- net TMS: now also D4.6 (K5), J3.4 (Pin_4)
- net IO0: now reaches U3.44 (MTDO)
- net IO0: now also D5.3 (K2), J3.1 (Pin_1)
- net EN_TCK renamed EN
- removed net IO0_TMS: D5.3 (K2), J3.1 (Pin_1), U3.42 (GPIO38)
- new net TCK: D4.4 (K3), J3.7 (Pin_7), U3.42 (GPIO38)
- no-connect marks 34 -> 32
Other:
- moved on the sheet: AE1, C15, C16, D10, D11, D4C, D4E, L1, R8, R9

Commit message: add type-c pull-down resistors
Parts:
- added R10, R11: 5.1k, Resistor_SMD:R_0402_1005Metric, symbol Device:R
Connections:
- net GND: now also R10.1, R11.1
- net at J2.A5 (CC1): now also R10.2
- net at J2.B5 (CC2): now also R11.2
- no-connect marks 32 -> 30
Changed lines of the file:
@@
 	1    0    0    -1
 $EndComp
-NoConn ~ 1700 2500
-NoConn ~ 1700 2600
 NoConn ~ 1700 3400
 NoConn ~ 1700 3500
@@
 $EndComp
 $Bitmap
-Pos 2500 2900
+Pos 2600 2950
 Scale 0.200000
 Data
@@
 Wire Notes Line
 	10950 1750 8150 1750
+$Comp
+L Device:R R10
+U 1 1 61E54E97
+P 1850 2500
+F 0 "R10" V 1800 2650 50  0000 L CNN
+F 1 "5.1k" V 1850 2400 50  0000 L CNN
+F 2 "Resistor_SMD:R_0402_1005Metric" V 1780 2500 50  0001 C CNN
+F 3 "~" H 1850 2500 50  0001 C CNN
+	1    1850 2500
+	0    1    1    0
+$EndComp
+$Comp
+L Device:R R11
+U 1 1 61E5695E
+P 1850 2600
+F 0 "R11" V 1800 2750 50  0000 L CNN
+F 1 "5.1k" V 1850 2500 50  0000 L CNN
+F 2 "Resistor_SMD:R_0402_1005Metric" V 1780 2600 50  0001 C CNN
+F 3 "~" H 1850 2600 50  0001 C CNN
+	1    1850 2600
+	0    1    1    0
+$EndComp
+$Comp
+L power:GND #PWR042
+U 1 1 61E570AA
+P 2150 2650
+F 0 "#PWR042" H 2150 2400 50  0001 C CNN
+F 1 "GND" H 2155 2477 50  0000 C CNN
+F 2 "" H 2150 2650 50  0001 C CNN
+F 3 "" H 2150 2650 50  0001 C CNN
+	1    2150 2650
+	1    0    0    -1
+$EndComp
+Wire Wire Line
+	2000 2500 2150 2500
+Wire Wire Line
+	2150 2500 2150 2600
+Wire Wire Line
+	2000 2600 2150 2600
+Connection ~ 2150 2600
+Wire Wire Line
+	2150 2600 2150 2650
 $EndSCHEMATC
