File: esp32s2-uart.sch (KiCad schematic (older format))
At the start: 51 parts, among them J1 USB_A, J2 USB_C_Receptacle_USB2.0, J3 Conn_02x05_Counter_Clockwise, SW1 SW_Push, U1 AMS1117-3.3, U2 USBLC6-2SC6, U3 ESP32-S2FH4, Y1 Crystal_GND24_Small

Commit message: v1.0
Connections:
- net IO0: now also D4.4 (K3), J3.7 (Pin_7), U3.42 (GPIO38); no longer D5.3 (K2), J3.1 (Pin_1), U3.44 (MTDO)
- net TCK: now also D5.3 (K2), J3.1 (Pin_1), U3.44 (MTDO); no longer D4.4 (K3), J3.7 (Pin_7), U3.42 (GPIO38)
Changed lines of the file:
@@
 Wire Wire Line
 	5700 1950 5800 1950
-Text Label 9000 3100 0    50   ~ 0
+Text Label 9950 3400 0    50   ~ 0
 IO0
 Text Label 9950 3300 0    50   ~ 0
@@
 Text Label 7350 3000 0    50   ~ 0
 EN
-Text Label 7350 2100 0    50   ~ 0
+Text Label 7350 2700 0    50   ~ 0
 IO0
 $Comp
@@
 Text Label 9000 3400 0    50   ~ 0
 TMS
-Text Label 9950 3400 0    50   ~ 0
+Text Label 9000 3100 0    50   ~ 0
 TCK
-Text Label 7350 2700 0    50   ~ 0
+Text Label 7350 2100 0    50   ~ 0
 TCK
 Wire Wire Line
